Commit message: Added scripts and launch files for keyboard control, applied controller plugin, and implementing ROS cmd_vel node
- Add keyboard_teleop.py (~/catkin_ws/src/ketg_description/scripts)
- Add keyboard_teleop.launch (~/catkin_ws/src/ketg_description/launch)
- Modify aibot_ketg_gazebo.xacro to apply controller plugin (~/catkin_ws/src/ketg_description/urdf)
- Implementing communication node for ROS topic cmd_vel (keyboard control topic)

File: ros1-gazebo-simulation-model/urdf/aibot_ketg_gazebo.xacro (robot description, xacro)
@@ -375,20 +375,20 @@
     <origin xyz="0.0 0.0 0.0" rpy="0 0 0"/>
   </joint>
-  <joint name="caster_back_left_joint" type="fixed">
+  <joint name="caster_back_left_joint" type="continuous">
     <parent link="0_Base_body_link"/>
     <child link="caster_back_left_link"/>
     <origin xyz="0.0 0.0 0.0" rpy="0 0 0"/>
   </joint>
-  <joint name="caster_back_right_joint" type="fixed">
+  <joint name="caster_back_right_joint" type="continuous">
     <parent link="0_Base_body_link"/>
     <child link="caster_back_right_link"/>
     <origin xyz="0.0 0.0 0.0" rpy="0 0 0"/>
   </joint>
-  <joint name="caster_front_left_joint" type="fixed">
+  <joint name="caster_front_left_joint" type="continuous">
     <parent link="0_Base_body_link"/>
     <child link="caster_front_left_link"/>
     <origin xyz="0.0 0.0 0.0" rpy="0 0 0"/>
   </joint>
-  <joint name="caster_front_right_joint" type="fixed">
+  <joint name="caster_front_right_joint" type="continuous">
     <parent link="0_Base_body_link"/>
     <child link="caster_front_right_link"/>
@@ -435,10 +435,10 @@
     <origin xyz="0.0 0.0 0.0" rpy="0 0 0"/>
   </joint>
-  <joint name="wheel_l_joint" type="fixed">
+  <joint name="wheel_l_joint" type="continuous">
     <parent link="0_Base_body_link"/>
     <child link="wheel_L_link"/>
     <origin xyz="0.0 0.0 0.0" rpy="0 0 0"/>
   </joint>
-  <joint name="wheel_r_joint" type="fixed">
+  <joint name="wheel_r_joint" type="continuous">
     <parent link="0_Base_body_link"/>
     <child link="wheel_R_link"/>
@@ -449,30 +449,23 @@
     <plugin name="gazebo_ros_control" filename="libgazebo_ros_control.so"/>
   </gazebo>
-  <gazebo>
-    <plugin name="joint_states" filename="libgazebo_ros_joint_state_publisher.so">
-      <joint_name>wheel_l_joint</joint_name>
-      <joint_name>wheel_r_joint</joint_name>
-      <updateRate>100</updateRate>
-    </plugin>
-    <plugin name="base_controller" filename="libgazebo_ros_diff_drive.so">
-      <commandTopic>cmd_vel</commandTopic>
-      <odometryTopic>robot/odom</odometryTopic>
-      <odometryFrame>odom</odometryFrame>
-      <odometrySource>world</odometrySource>
-      <publishOdomTF>true</publishOdomTF>
-      <robotBaseFrame>0_Base_body_link</robotBaseFrame>
-      <publishWheelTF>false</publishWheelTF>
-      <publishTf>true</publishTf>
-      <publishWheelJointState>true</publishWheelJointState>
-      <legacyMode>false</legacyMode>
-      <updateRate>30</updateRate>
-      <leftJoint>wheel_l_joint</leftJoint>
-      <rightJoint>wheel_r_joint</rightJoint>
-      <wheelSeparation>0.347</wheelSeparation>
-      <wheelDiameter>0.130</wheelDiameter>
-      <wheelAcceleration>1</wheelAcceleration>
-      <wheelTorque>10</wheelTorque>
-      <rosDebugLevel>na</rosDebugLevel>
-    </plugin>
-  </gazebo>
+<gazebo>
+  <plugin name="gazebo_ros_diff_drive" filename="libgazebo_ros_diff_drive.so">
+    <commandTopic>cmd_vel</commandTopic>
+    <odometryTopic>odom</odometryTopic>
+    <odometryFrame>odom</odometryFrame>
+    <robotBaseFrame>base_link</robotBaseFrame>
+    <publishOdomTF>true</publishOdomTF>
+    <publishWheelTF>false</publishWheelTF>
+    <publishTf>true</publishTf>
+    <publishWheelJointState>true</publishWheelJointState>
+    <legacyMode>false</legacyMode>
+    <updateRate>30</updateRate>
+    <leftJoint>wheel_L_joint</leftJoint>
+    <rightJoint>wheel_R_joint</rightJoint>
+    <wheelSeparation>0.347</wheelSeparation>
+    <wheelDiameter>0.130</wheelDiameter>
+    <wheelAcceleration>1</wheelAcceleration>
+    <wheelTorque>10</wheelTorque>
+  </plugin>
+</gazebo>
 </robot>
